Commit message: change of file structure like in ros2_control_demos

File: omni_car/description/urdf/wheel.xacro (robot description, xacro)
@@ -1,6 +1,6 @@
 <?xml version="1.0"?>
 <robot xmlns:xacro="http://wiki.ros.org/xacro">
-    <xacro:macro name="wheel" params="wheel_name is_right wheel_x_offset wheel_y_offset wheel_z_offset">
-        <link name="wheel_${wheel_name}">
+    <xacro:macro name="wheel" params="wheel_name is_right wheel_x_offset wheel_y_offset wheel_z_offset prefix">
+        <link name="${prefix}wheel_${wheel_name}">
             <inertial>
                 <origin xyz="0 0 0" rpy="0 0 0" />
@@ -12,22 +12,20 @@
                 <geometry>
                     <xacro:if value="${is_right}">
-                        <mesh filename="file://$(find omni_car_description)/meshes/wheel_r.dae" />
+                        <mesh filename="file://$(find omni_car)/meshes/wheel_r.dae" />
                     </xacro:if>
                     <xacro:unless value="${is_right}">
-                        <mesh filename="file://$(find omni_car_description)/meshes/wheel_l.dae" />
+                        <mesh filename="file://$(find omni_car)/meshes/wheel_l.dae" />
                     </xacro:unless>
                 </geometry>
-                <material name="">
-                    <color rgba="0.77 0 1 1" />
-                </material>
+                <material name="yellow"/>
             </visual>
             <collision>
                 <origin xyz="0 0 0" rpy="0 0 0" />
                 <geometry>
-                    <cylinder radius="0.0" length="0.0"/>
+                    <cylinder radius="0.0001" length="0.0001"/>
                 </geometry>
             </collision>
         </link>
-        <link name="wheel_${wheel_name}_force_transform">
+        <link name="${prefix}wheel_${wheel_name}_force_transform">
             <inertial>
                 <origin xyz="0 0 0" rpy="0 0 0" />
@@ -38,5 +36,5 @@
                 <origin xyz="0 0 0" rpy="0 0 0" />
                 <geometry>
-                    <cylinder radius="0.0" length="0.0"/>
+                    <cylinder radius="0.0001" length="0.0001"/>
                 </geometry>
             </visual>
@@ -48,14 +46,14 @@
             </collision>
         </link>
-        <joint name="wheel_${wheel_name}_joint" type="continuous">
-            <parent link="frame" />
-            <child link="wheel_${wheel_name}" />
+        <joint name="${prefix}wheel_${wheel_name}_joint" type="continuous">
+            <parent link="${prefix}frame" />
+            <child link="${prefix}wheel_${wheel_name}" />
             <axis xyz="0 0 1" />
             <origin xyz="${wheel_x_offset} ${wheel_y_offset} ${wheel_z_offset}" rpy="${-pi/2} 0 0"/>
             <limit velocity="15.0" effort="30"/>
         </joint>
-        <joint name="wheel_${wheel_name}_joint_force_transform" type="continuous">
-            <parent link="frame"/>
-            <child link="wheel_${wheel_name}_force_transform"/>
+        <joint name="${prefix}wheel_${wheel_name}_joint_force_transform" type="continuous">
+            <parent link="${prefix}frame"/>
+            <child link="${prefix}wheel_${wheel_name}_force_transform"/>
             <xacro:if value="${is_right}">
                 <origin xyz="${wheel_x_offset} ${wheel_y_offset} ${wheel_z_offset}" rpy="${-pi/2} 0 ${pi/4}"/> <!-- 45 deg rotate -->
@@ -65,21 +63,15 @@
             </xacro:unless>
             <axis xyz="0 0 1"/>
-            <mimic joint="wheel_${wheel_name}_joint" multiplier="1.0"/>
+            <mimic joint="${prefix}wheel_${wheel_name}_joint" multiplier="1.0"/>
         </joint>
-        <transmission name="${wheel_name}_trans">
+        <transmission name="${prefix}${wheel_name}_trans">
             <type>transmission_interface/SimpleTransmission</type>
-            <joint name="wheel_${wheel_name}_joint">
+            <joint name="${prefix}wheel_${wheel_name}_joint">
                 <hardwareInterface>VelocityJointInterface</hardwareInterface>
             </joint>
-            <actuator name="${wheel_name}_motor">
+            <actuator name="${prefix}${wheel_name}_motor">
                 <mechanicalReduction>1</mechanicalReduction>
             </actuator>
         </transmission>
-        <!-- <ros2_control>
-            <joint name="wheel_${wheel_name}_joint">
-                <command_interface name="velocity"/>
-                <state_interface name="velocity"/>
-            </joint>
-        </ros2_control> -->
     </xacro:macro>
 </robot>
