Commit message: changed wheel order

File: omni_car/description/urdf/omni_car_description.xacro (robot description, xacro)
@@ -31,10 +31,10 @@
   </joint>
   <xacro:property name="wheel_x_offset" value="0.081"/>
-  <xacro:property name="wheel_y_offset" value="0.098"/>
+  <xacro:property name="wheel_y_offset" value="0.081"/>
   <xacro:property name="wheel_z_offset" value="-0.02"/>
-  <xacro:wheel wheel_name="front_left" is_right="false" wheel_x_offset="${wheel_x_offset}" wheel_y_offset="${wheel_y_offset}" wheel_z_offset="${wheel_z_offset}" prefix="${prefix}"/>
-  <xacro:wheel wheel_name="front_right" is_right="true" wheel_x_offset="${wheel_x_offset}" wheel_y_offset="${-wheel_y_offset}" wheel_z_offset="${wheel_z_offset}" prefix="${prefix}"/>
-  <xacro:wheel wheel_name="rear_left" is_right="false" wheel_x_offset="${-wheel_x_offset}" wheel_y_offset="${wheel_y_offset}" wheel_z_offset="${wheel_z_offset}" prefix="${prefix}"/>
-  <xacro:wheel wheel_name="rear_right" is_right="true" wheel_x_offset="${-wheel_x_offset}" wheel_y_offset="${-wheel_y_offset}" wheel_z_offset="${wheel_z_offset}" prefix="${prefix}"/>
+  <xacro:wheel wheel_name="front_left" is_right="false" is_front="true" wheel_x_offset="${wheel_x_offset}" wheel_y_offset="${wheel_y_offset}" wheel_z_offset="${wheel_z_offset}" prefix="${prefix}"/>
+  <xacro:wheel wheel_name="front_right" is_right="true" is_front="true" wheel_x_offset="${wheel_x_offset}" wheel_y_offset="${-wheel_y_offset}" wheel_z_offset="${wheel_z_offset}" prefix="${prefix}"/>
+  <xacro:wheel wheel_name="rear_left" is_right="false" is_front="false" wheel_x_offset="${-wheel_x_offset}" wheel_y_offset="${wheel_y_offset}" wheel_z_offset="${wheel_z_offset}" prefix="${prefix}"/>
+  <xacro:wheel wheel_name="rear_right" is_right="true" is_front="false" wheel_x_offset="${-wheel_x_offset}" wheel_y_offset="${-wheel_y_offset}" wheel_z_offset="${wheel_z_offset}" prefix="${prefix}"/>
   </xacro:macro>
 </robot>

File: omni_car/description/urdf/wheel.xacro (robot description, xacro)
@@ -1,5 +1,5 @@
 <?xml version="1.0"?>
 <robot xmlns:xacro="http://wiki.ros.org/xacro">
-    <xacro:macro name="wheel" params="wheel_name is_right wheel_x_offset wheel_y_offset wheel_z_offset prefix">
+    <xacro:macro name="wheel" params="wheel_name is_right is_front wheel_x_offset wheel_y_offset wheel_z_offset prefix">
         <link name="${prefix}wheel_${wheel_name}">
             <inertial>
@@ -9,11 +9,13 @@
             </inertial>
             <visual>
-                <origin xyz="0 0 0" rpy="0 0 0" />
+                <origin xyz="0 0 0" rpy="${-pi/2} 0 0" />
                 <geometry>
-                    <xacro:if value="${is_right}">
-                        <mesh filename="file://$(find omni_car)/meshes/wheel_r.dae" />
+                    <!-- <xacro:if value="${is_right}"> -->
+                    <xacro:if value="${(is_right and is_front) or (not is_right and not is_front)}">
+                        <mesh filename="file://$(find omni_car)/meshes/wheel_set2.dae" />
                     </xacro:if>
-                    <xacro:unless value="${is_right}">
-                        <mesh filename="file://$(find omni_car)/meshes/wheel_l.dae" />
+                    <!-- <xacro:unless value="${is_right}"> -->
+                    <xacro:unless value="${(is_right and is_front) or (not is_right and not is_front)}">
+                        <mesh filename="file://$(find omni_car)/meshes/wheel_set1.dae" />
                     </xacro:unless>
                 </geometry>
@@ -36,6 +38,6 @@
                 <origin xyz="0 0 0" rpy="0 0 0" />
                 <geometry>
-                    <!-- <cylinder radius="0.0001" length="0.0001"/> -->
-                    <cylinder radius="0.03" length="0.05"/>
+                    <cylinder radius="0.0001" length="0.0001"/>
+                    <!-- <cylinder radius="0.03" length="0.02"/> -->
                 </geometry>
             </visual>
@@ -43,5 +45,5 @@
                 <origin xyz="0 0 0" rpy="0 0 0" />
                 <geometry>
-                    <cylinder radius="0.03" length="0.05"/>
+                    <cylinder radius="0.03" length="0.02"/>
                 </geometry>
             </collision>
@@ -57,9 +59,9 @@
             <parent link="${prefix}frame"/>
             <child link="${prefix}wheel_${wheel_name}_force_transform"/>
-            <xacro:if value="${is_right}">
+            <xacro:if value="${(is_right and is_front) or (not is_right and not is_front)}">
                 <origin xyz="${wheel_x_offset} ${wheel_y_offset} ${wheel_z_offset}" rpy="${-pi/2} 0 ${pi/4}"/> <!-- 45 deg rotate -->
             </xacro:if>
-            <xacro:unless value="${is_right}">
-                <origin xyz="${wheel_x_offset} ${wheel_y_offset} ${wheel_z_offset}" rpy="${-pi/2} 0 ${-pi/4}"/> <!-- 45 deg rotate -->
+            <xacro:unless value="${(is_right and is_front) or (not is_right and not is_front)}">
+                <origin xyz="${wheel_x_offset} ${wheel_y_offset} ${wheel_z_offset}" rpy="${-pi/2} 0 ${-pi/4}"/> <!-- -45 deg rotate -->
             </xacro:unless>
             <axis xyz="0 0 1"/>
