Commit message: imu and lidar in model (gazebo todo)

File: omni_car/description/urdf/omni_car.xacro (robot description, xacro)
@@ -2,5 +2,5 @@
 <robot name="omni_car" xmlns:xacro="http://www.ros.org/wiki/xacro">
   <xacro:arg name="prefix" default=""/>
-  <xacro:include filename="$(find omni_car)/urdf/omni_car_description.xacro"/>
+  <xacro:include filename="$(find omni_car)/urdf/omni_car_description.urdf.xacro"/>
   <xacro:include filename="$(find omni_car)/gazebo/omni_car.gazebo.xacro"/>
   <xacro:include filename="$(find omni_car)/ros2_control/omni_car.ros2_control.xacro"/>

File: omni_car/description/urdf/omni_car_description.urdf.xacro (robot description, xacro)
@@ -3,5 +3,7 @@
   <xacro:macro name="omni_car" params="prefix">
   <xacro:include filename="$(find omni_car)/urdf/omni_car.materials.xacro"/>
-  <xacro:include filename="$(find omni_car)/urdf/wheel.xacro"/>
+  <xacro:include filename="$(find omni_car)/urdf/wheel.urdf.xacro"/>
+  <xacro:include filename="$(find omni_car)/urdf/imu.urdf.xacro"/>
+  <xacro:include filename="$(find omni_car)/urdf/lidar.urdf.xacro"/>
   <link name="${prefix}base_link"/>
   <link name="${prefix}frame">
@@ -37,4 +39,10 @@
   <xacro:wheel wheel_site="rear_left" wheel_x_offset="${-wheel_x_offset}" wheel_y_offset="${wheel_y_offset}" wheel_z_offset="${wheel_z_offset}" prefix="${prefix}"/>
   <xacro:wheel wheel_site="rear_right" wheel_x_offset="${-wheel_x_offset}" wheel_y_offset="${-wheel_y_offset}" wheel_z_offset="${wheel_z_offset}" prefix="${prefix}"/>
+  <xacro:imu name="imu" prefix="${prefix}">
+    <origin xyz="0 0 -0.001" rpy="0 0 0"/>
+  </xacro:imu>
+  <xacro:lidar name="lidar" prefix="${prefix}">
+    <origin xyz="-0.042 0 0.005" rpy="0 0 0"/>
+  </xacro:lidar>
   </xacro:macro>
 </robot>
