Commit message: kinect camera model - todo gazebo, joint_state_publisher in gazebo launch

File: omni_car/description/urdf/imu.urdf.xacro (robot description, xacro)
@@ -2,5 +2,5 @@
 <robot xmlns:xacro="http://wiki.ros.org/xacro">
   <xacro:property name="imu_size" value="0.002" />
-  <xacro:macro name="imu" params="name prefix *origin">
+  <xacro:macro name="imu" params="name parent_frame prefix *origin">
     <link name="${prefix}${name}_link">
       <visual>
@@ -14,5 +14,5 @@
     <joint name="${prefix}${name}_joint" type="fixed">
       <xacro:insert_block name="origin" />
-      <parent link="${prefix}frame"/>
+      <parent link="${parent_frame}"/>
       <child link="${prefix}${name}_link"/>
     </joint>

File: omni_car/description/urdf/lidar.urdf.xacro (robot description, xacro)
@@ -3,7 +3,7 @@
   <xacro:property name="lidar_base_size_x" value="0.1" />
   <xacro:property name="lidar_base_size_y" value="0.08" />
-  <xacro:property name="lidar_base_size_z" value="0.002" />
-  <xacro:property name="beam_z" value="0.045" />
-  <xacro:macro name="lidar" params="name prefix *origin">
+  <xacro:property name="lidar_base_size_z" value="0.035" />
+  <xacro:property name="beam_z" value="0.06" />
+  <xacro:macro name="lidar" params="name parent_frame prefix *origin">
     <link name="${prefix}${name}_base_link">
       <visual>
@@ -27,5 +27,5 @@
     <joint name="${prefix}${name}_base_joint" type="fixed">
       <xacro:insert_block name="origin" />
-      <parent link="${prefix}frame"/>
+      <parent link="${parent_frame}"/>
       <child link="${prefix}${name}_base_link"/>
     </joint>

File: omni_car/description/urdf/omni_car_description.urdf.xacro (robot description, xacro)
@@ -6,13 +6,12 @@
   <xacro:include filename="$(find omni_car)/urdf/imu.urdf.xacro"/>
   <xacro:include filename="$(find omni_car)/urdf/lidar.urdf.xacro"/>
+  <xacro:include filename="$(find omni_car)/urdf/kinect.urdf.xacro"/>
   <link name="${prefix}base_link"/>
   <link name="${prefix}frame">
     <inertial>
-      <origin xyz="0 0 0" rpy="0 0 0" />
-      <mass value="200.0" />
+      <mass value="20.0" />
       <inertia ixx="0.02" ixy="0.0" ixz="0.0" iyy="0.02" iyz="0.0" izz="0.02" />
     </inertial>
     <visual>
-      <origin xyz="0 0 0" rpy="0 0 0" />
       <geometry>
         <mesh filename="file://$(find omni_car)/meshes/base_link.dae" />
@@ -21,5 +20,4 @@
     </visual>
     <collision>
-      <origin xyz="0 0 0" rpy="0 0 0" />
       <geometry>
         <box size="0.23 0.1 0.01"/>
@@ -39,10 +37,13 @@
   <xacro:wheel wheel_site="rear_left" wheel_x_offset="${-wheel_x_offset}" wheel_y_offset="${wheel_y_offset}" wheel_z_offset="${wheel_z_offset}" prefix="${prefix}"/>
   <xacro:wheel wheel_site="rear_right" wheel_x_offset="${-wheel_x_offset}" wheel_y_offset="${-wheel_y_offset}" wheel_z_offset="${wheel_z_offset}" prefix="${prefix}"/>
-  <xacro:imu name="imu" prefix="${prefix}">
+  <xacro:imu name="imu" parent_frame="${prefix}frame" prefix="${prefix}">
     <origin xyz="0 0 -0.001" rpy="0 0 0"/>
   </xacro:imu>
-  <xacro:lidar name="lidar" prefix="${prefix}">
-    <origin xyz="-0.042 0 0.005" rpy="0 0 0"/>
+  <xacro:lidar name="lidar" parent_frame="${prefix}frame" prefix="${prefix}">
+    <origin xyz="-0.042 0 0.0215" rpy="0 0 0"/>
   </xacro:lidar>
+  <xacro:kinect name="kinect" parent_frame="${prefix}frame" prefix="${prefix}">
+    <origin xyz="0.1 0 0.055" rpy="0 0 0"/>
+  </xacro:kinect>
   </xacro:macro>
 </robot>
