Commit message: gz physics engine from DART to Bullet

File: omni_car/description/gazebo/omni_car.gazebo.xacro (robot description, xacro)
@@ -7,12 +7,26 @@
       </plugin>
     </gazebo>
-    <!-- <gazebo reference="${prefix}base_link">
+    <gazebo reference="${prefix}base_link">
       <material>Gazebo/Orange</material>
     </gazebo>
-    <gazebo reference="${prefix}link1">
-      <mu1>0.2</mu1>
-      <mu2>0.2</mu2>
-      <material>Gazebo/Yellow</material>
-    </gazebo> -->
+    <!-- Visual and collision properties for wheels -->
+    <xacro:property name="wheel_mu1" value="0.8"/>
+    <xacro:property name="wheel_mu2" value="0.7"/>
+    <xacro:property name="wheel_material" value="Gazebo/Yellow"/>
+    <xacro:macro name="wheel_properties" params="wheel_name">
+      <gazebo reference="${prefix}${wheel_name}">
+        <mu1>${wheel_mu1}</mu1>
+        <mu2>${wheel_mu2}</mu2>
+        <material>${wheel_material}</material>
+      </gazebo>
+      <gazebo reference="${prefix}${wheel_name}_force_transform">
+        <mu1>${wheel_mu1}</mu1>
+        <mu2>${wheel_mu2}</mu2>
+      </gazebo>
+    </xacro:macro>
+    <xacro:wheel_properties wheel_name="wheel_front_left"/>
+    <xacro:wheel_properties wheel_name="wheel_front_right"/>
+    <xacro:wheel_properties wheel_name="wheel_rear_left"/>
+    <xacro:wheel_properties wheel_name="wheel_rear_right"/>
   </xacro:macro>
 </robot>

File: omni_car/description/urdf/wheel.xacro (robot description, xacro)
@@ -36,5 +36,6 @@
                 <origin xyz="0 0 0" rpy="0 0 0" />
                 <geometry>
-                    <cylinder radius="0.0001" length="0.0001"/>
+                    <!-- <cylinder radius="0.0001" length="0.0001"/> -->
+                    <cylinder radius="0.03" length="0.05"/>
                 </geometry>
             </visual>

Commit message: joy steering

File: omni_car/description/gazebo/omni_car.gazebo.xacro (robot description, xacro)
@@ -11,6 +11,6 @@
     </gazebo>
     <!-- Visual and collision properties for wheels -->
-    <xacro:property name="wheel_mu1" value="0.8"/>
-    <xacro:property name="wheel_mu2" value="0.7"/>
+    <xacro:property name="wheel_mu1" value="0.2"/>
+    <xacro:property name="wheel_mu2" value="0.1"/>
     <xacro:property name="wheel_material" value="Gazebo/Yellow"/>
     <xacro:macro name="wheel_properties" params="wheel_name">

File: omni_car/description/urdf/omni_car_description.xacro (robot description, xacro)
@@ -8,5 +8,5 @@
     <inertial>
       <origin xyz="0 0 0" rpy="0 0 0" />
-      <mass value="2.0" />
+      <mass value="200.0" />
       <inertia ixx="0.02" ixy="0.0" ixz="0.0" iyy="0.02" iyz="0.0" izz="0.02" />
     </inertial>
@@ -21,5 +21,5 @@
       <origin xyz="0 0 0" rpy="0 0 0" />
       <geometry>
-        <box size="0.23 0.13 0.01"/>
+        <box size="0.23 0.1 0.01"/>
       </geometry>
     </collision>

File: omni_car/description/urdf/wheel.xacro (robot description, xacro)
@@ -39,5 +39,4 @@
                 <geometry>
                     <cylinder radius="0.0001" length="0.0001"/>
-                    <!-- <cylinder radius="0.03" length="0.02"/> -->
                 </geometry>
             </visual>

Commit message: into gazebo plugun, build ok, not working yet

File: omni_car/description/gazebo/omni_car.gazebo.xacro (robot description, xacro)
@@ -10,7 +10,13 @@
       <material>Gazebo/Orange</material>
     </gazebo>
+    <!-- Add the force plugin here -->
+    <gazebo>
+      <plugin filename="force_plugin" name="force_plugin::ForcePlugin">
+        <bodyName>${prefix}base_link</bodyName>
+      </plugin>
+    </gazebo>
     <!-- Visual and collision properties for wheels -->
-    <xacro:property name="wheel_mu1" value="0.2"/>
-    <xacro:property name="wheel_mu2" value="0.1"/>
+    <xacro:property name="wheel_mu1" value="0.0"/>
+    <xacro:property name="wheel_mu2" value="0.0"/>
     <xacro:property name="wheel_material" value="Gazebo/Yellow"/>
     <xacro:macro name="wheel_properties" params="wheel_name">

Commit message: Abandoning the idea of 45-degree wheel collisions, plugin works

File: omni_car/description/gazebo/omni_car.gazebo.xacro (robot description, xacro)
@@ -14,4 +14,5 @@
       <plugin filename="force_plugin" name="force_plugin::ForcePlugin">
         <bodyName>${prefix}base_link</bodyName>
+        <cmdTopic>omni_car_controller/cmd_vel</cmdTopic>
       </plugin>
     </gazebo>
@@ -26,8 +27,8 @@
         <material>${wheel_material}</material>
       </gazebo>
-      <gazebo reference="${prefix}${wheel_name}_force_transform">
+      <!-- <gazebo reference="${prefix}${wheel_name}_force_transform">
         <mu1>${wheel_mu1}</mu1>
         <mu2>${wheel_mu2}</mu2>
-      </gazebo>
+      </gazebo> -->
     </xacro:macro>
     <xacro:wheel_properties wheel_name="wheel_front_left"/>

File: omni_car/description/urdf/wheel.xacro (robot description, xacro)
@@ -25,9 +25,10 @@
                 <origin xyz="0 0 0" rpy="0 0 0" />
                 <geometry>
-                    <cylinder radius="0.0001" length="0.0001"/>
+                    <!-- <cylinder radius="0.0001" length="0.0001"/> -->
+                    <cylinder radius="0.03" length="0.02"/>
                 </geometry>
             </collision>
         </link>
-        <link name="${prefix}wheel_${wheel_name}_force_transform">
+        <!-- <link name="${prefix}wheel_${wheel_name}_force_transform">
             <inertial>
                 <origin xyz="0 0 0" rpy="0 0 0" />
@@ -47,5 +48,5 @@
                 </geometry>
             </collision>
-        </link>
+        </link> -->
         <joint name="${prefix}wheel_${wheel_name}_joint" type="continuous">
             <parent link="${prefix}frame" />
@@ -55,16 +56,16 @@
             <limit velocity="15.0" effort="30"/>
         </joint>
-        <joint name="${prefix}wheel_${wheel_name}_joint_force_transform" type="continuous">
+        <!-- <joint name="${prefix}wheel_${wheel_name}_joint_force_transform" type="continuous">
             <parent link="${prefix}frame"/>
             <child link="${prefix}wheel_${wheel_name}_force_transform"/>
             <xacro:if value="${(is_right and is_front) or (not is_right and not is_front)}">
-                <origin xyz="${wheel_x_offset} ${wheel_y_offset} ${wheel_z_offset}" rpy="${-pi/2} 0 ${pi/4}"/> <!-- 45 deg rotate -->
+                <origin xyz="${wheel_x_offset} ${wheel_y_offset} ${wheel_z_offset}" rpy="${-pi/2} 0 ${pi/4}"/>  45 deg rotate
             </xacro:if>
             <xacro:unless value="${(is_right and is_front) or (not is_right and not is_front)}">
-                <origin xyz="${wheel_x_offset} ${wheel_y_offset} ${wheel_z_offset}" rpy="${-pi/2} 0 ${-pi/4}"/> <!-- -45 deg rotate -->
+                <origin xyz="${wheel_x_offset} ${wheel_y_offset} ${wheel_z_offset}" rpy="${-pi/2} 0 ${-pi/4}"/>  -45 deg rotate
             </xacro:unless>
             <axis xyz="0 0 1"/>
             <mimic joint="${prefix}wheel_${wheel_name}_joint" multiplier="1.0"/>
-        </joint>
+        </joint> -->
         <transmission name="${prefix}${wheel_name}_trans">
             <type>transmission_interface/SimpleTransmission</type>

Commit message: model improvement

File: omni_car/description/gazebo/omni_car.gazebo.xacro (robot description, xacro)
@@ -17,5 +17,5 @@
       </plugin>
     </gazebo>
-    <!-- Visual and collision properties for wheels -->
+    <!-- Properties for wheels -->
     <xacro:property name="wheel_mu1" value="0.0"/>
     <xacro:property name="wheel_mu2" value="0.0"/>
@@ -27,8 +27,4 @@
         <material>${wheel_material}</material>
       </gazebo>
-      <!-- <gazebo reference="${prefix}${wheel_name}_force_transform">
-        <mu1>${wheel_mu1}</mu1>
-        <mu2>${wheel_mu2}</mu2>
-      </gazebo> -->
     </xacro:macro>
     <xacro:wheel_properties wheel_name="wheel_front_left"/>

File: omni_car/description/urdf/omni_car_description.xacro (robot description, xacro)
@@ -30,11 +30,11 @@
     <origin xyz="0 0 0" rpy="0 0 0"/>
   </joint>
-  <xacro:property name="wheel_x_offset" value="0.081"/>
-  <xacro:property name="wheel_y_offset" value="0.081"/>
-  <xacro:property name="wheel_z_offset" value="-0.02"/>
-  <xacro:wheel wheel_name="front_left" is_right="false" is_front="true" wheel_x_offset="${wheel_x_offset}" wheel_y_offset="${wheel_y_offset}" wheel_z_offset="${wheel_z_offset}" prefix="${prefix}"/>
-  <xacro:wheel wheel_name="front_right" is_right="true" is_front="true" wheel_x_offset="${wheel_x_offset}" wheel_y_offset="${-wheel_y_offset}" wheel_z_offset="${wheel_z_offset}" prefix="${prefix}"/>
-  <xacro:wheel wheel_name="rear_left" is_right="false" is_front="false" wheel_x_offset="${-wheel_x_offset}" wheel_y_offset="${wheel_y_offset}" wheel_z_offset="${wheel_z_offset}" prefix="${prefix}"/>
-  <xacro:wheel wheel_name="rear_right" is_right="true" is_front="false" wheel_x_offset="${-wheel_x_offset}" wheel_y_offset="${-wheel_y_offset}" wheel_z_offset="${wheel_z_offset}" prefix="${prefix}"/>
+  <xacro:property name="wheel_x_offset" value="0.08"/>
+  <xacro:property name="wheel_y_offset" value="0.078"/>
+  <xacro:property name="wheel_z_offset" value="-0.018"/>
+  <xacro:wheel wheel_site="front_left" wheel_x_offset="${wheel_x_offset}" wheel_y_offset="${wheel_y_offset}" wheel_z_offset="${wheel_z_offset}" prefix="${prefix}"/>
+  <xacro:wheel wheel_site="front_right" wheel_x_offset="${wheel_x_offset}" wheel_y_offset="${-wheel_y_offset}" wheel_z_offset="${wheel_z_offset}" prefix="${prefix}"/>
+  <xacro:wheel wheel_site="rear_left" wheel_x_offset="${-wheel_x_offset}" wheel_y_offset="${wheel_y_offset}" wheel_z_offset="${wheel_z_offset}" prefix="${prefix}"/>
+  <xacro:wheel wheel_site="rear_right" wheel_x_offset="${-wheel_x_offset}" wheel_y_offset="${-wheel_y_offset}" wheel_z_offset="${wheel_z_offset}" prefix="${prefix}"/>
   </xacro:macro>
 </robot>

File: omni_car/description/urdf/wheel.xacro (robot description, xacro)
@@ -1,6 +1,6 @@
 <?xml version="1.0"?>
 <robot xmlns:xacro="http://wiki.ros.org/xacro">
-    <xacro:macro name="wheel" params="wheel_name is_right is_front wheel_x_offset wheel_y_offset wheel_z_offset prefix">
-        <link name="${prefix}wheel_${wheel_name}">
+    <xacro:macro name="wheel" params="wheel_site wheel_x_offset wheel_y_offset wheel_z_offset prefix">
+        <link name="${prefix}wheel_${wheel_site}">
             <inertial>
                 <origin xyz="0 0 0" rpy="0 0 0" />
@@ -11,34 +11,7 @@
                 <origin xyz="0 0 0" rpy="${-pi/2} 0 0" />
                 <geometry>
-                    <!-- <xacro:if value="${is_right}"> -->
-                    <xacro:if value="${(is_right and is_front) or (not is_right and not is_front)}">
-                        <mesh filename="file://$(find omni_car)/meshes/wheel_set2.dae" />
-                    </xacro:if>
-                    <!-- <xacro:unless value="${is_right}"> -->
-                    <xacro:unless value="${(is_right and is_front) or (not is_right and not is_front)}">
-                        <mesh filename="file://$(find omni_car)/meshes/wheel_set1.dae" />
-                    </xacro:unless>
+                    <mesh filename="file://$(find omni_car)/meshes/wheel_${wheel_site}.dae" />
                 </geometry>
                 <material name="yellow"/>
-            </visual>
-            <collision>
-                <origin xyz="0 0 0" rpy="0 0 0" />
-                <geometry>
-                    <!-- <cylinder radius="0.0001" length="0.0001"/> -->
-                    <cylinder radius="0.03" length="0.02"/>
-                </geometry>
-            </collision>
-        </link>
-        <!-- <link name="${prefix}wheel_${wheel_name}_force_transform">
-            <inertial>
-                <origin xyz="0 0 0" rpy="0 0 0" />
-                <mass value="0.3" />
-                <inertia ixx="0.02" ixy="0.0" ixz="0.0" iyy="0.02" iyz="0.0" izz="0.02" />
-            </inertial>
-            <visual>
-                <origin xyz="0 0 0" rpy="0 0 0" />
-                <geometry>
-                    <cylinder radius="0.0001" length="0.0001"/>
-                </geometry>
             </visual>
             <collision>
@@ -48,30 +21,18 @@
                 </geometry>
             </collision>
-        </link> -->
-        <joint name="${prefix}wheel_${wheel_name}_joint" type="continuous">
+        </link>
+        <joint name="${prefix}wheel_${wheel_site}_joint" type="continuous">
             <parent link="${prefix}frame" />
-            <child link="${prefix}wheel_${wheel_name}" />
+            <child link="${prefix}wheel_${wheel_site}" />
             <axis xyz="0 0 1" />
             <origin xyz="${wheel_x_offset} ${wheel_y_offset} ${wheel_z_offset}" rpy="${-pi/2} 0 0"/>
             <limit velocity="15.0" effort="30"/>
         </joint>
-        <!-- <joint name="${prefix}wheel_${wheel_name}_joint_force_transform" type="continuous">
-            <parent link="${prefix}frame"/>
-            <child link="${prefix}wheel_${wheel_name}_force_transform"/>
-            <xacro:if value="${(is_right and is_front) or (not is_right and not is_front)}">
-                <origin xyz="${wheel_x_offset} ${wheel_y_offset} ${wheel_z_offset}" rpy="${-pi/2} 0 ${pi/4}"/>  45 deg rotate
-            </xacro:if>
-            <xacro:unless value="${(is_right and is_front) or (not is_right and not is_front)}">
-                <origin xyz="${wheel_x_offset} ${wheel_y_offset} ${wheel_z_offset}" rpy="${-pi/2} 0 ${-pi/4}"/>  -45 deg rotate
-            </xacro:unless>
-            <axis xyz="0 0 1"/>
-            <mimic joint="${prefix}wheel_${wheel_name}_joint" multiplier="1.0"/>
-        </joint> -->
-        <transmission name="${prefix}${wheel_name}_trans">
+        <transmission name="${prefix}${wheel_site}_trans">
             <type>transmission_interface/SimpleTransmission</type>
-            <joint name="${prefix}wheel_${wheel_name}_joint">
+            <joint name="${prefix}wheel_${wheel_site}_joint">
                 <hardwareInterface>VelocityJointInterface</hardwareInterface>
             </joint>
-            <actuator name="${prefix}${wheel_name}_motor">
+            <actuator name="${prefix}${wheel_site}_motor">
                 <mechanicalReduction>1</mechanicalReduction>
             </actuator>

Commit message: imu works

File: omni_car/description/gazebo/omni_car.gazebo.xacro (robot description, xacro)
@@ -1,23 +1,22 @@
 <robot xmlns:xacro="http://ros.org/wiki/xacro">
   <xacro:macro name="omni_car_gazebo" params="prefix">
-    <!-- ros_control plugin -->
     <gazebo>
+      <!-- ros2_control plugin -->
       <plugin filename="gz_ros2_control-system" name="gz_ros2_control::GazeboSimROS2ControlPlugin">
         <parameters>$(find omni_car)/config/omni_car_controllers.yaml</parameters>
       </plugin>
+      <!-- Sensors plugins -->
       <plugin filename="gz-sim-sensors-system" name="gz::sim::systems::Sensors">
         <render_engine>ogre2</render_engine>
       </plugin>
       <plugin filename="gz-sim-imu-system" name="gz::sim::systems::Imu"/>
-    </gazebo>
-    <gazebo reference="${prefix}base_link">
-      <material>Gazebo/Orange</material>
-    </gazebo>
-    <!-- Add the force plugin here -->
-    <gazebo>
+      <!-- Force plugin (solution to the problem mecanum wheels) -->
       <plugin filename="force_plugin" name="force_plugin::ForcePlugin">
         <bodyName>${prefix}base_link</bodyName>
         <cmdTopic>omni_car_controller/cmd_vel</cmdTopic>
       </plugin>
+    </gazebo>
+    <gazebo reference="${prefix}base_link">
+      <material>Gazebo/Orange</material>
     </gazebo>
     <!-- Properties for wheels -->
@@ -36,4 +35,6 @@
     <xacro:wheel_properties wheel_name="wheel_rear_left"/>
     <xacro:wheel_properties wheel_name="wheel_rear_right"/>
+    <!-- _____Sensors_____ -->
+    <!-- Lidar -->
     <gazebo reference="${prefix}lidar_beam_link" >
       <sensor name="lidar" type="gpu_lidar">
@@ -67,12 +68,13 @@
       </sensor>
     </gazebo>
+    <!-- IMU -->
     <gazebo reference="${prefix}imu_link" >
-        <sensor name="imu" type="imu">
-          <always_on>1</always_on>
-          <update_rate>100</update_rate>
-          <visualize>true</visualize>
-          <topic>imu</topic>
-          <enable_metrics>true</enable_metrics>
-        </sensor>
+      <sensor name="imu" type="imu">
+        <always_on>1</always_on>
+        <update_rate>100</update_rate>
+        <visualize>true</visualize>
+        <topic>imu</topic>
+        <enable_metrics>true</enable_metrics>
+      </sensor>
     </gazebo>
   </xacro:macro>

Commit message: rgb+depth cameras

File: omni_car/description/gazebo/omni_car.gazebo.xacro (robot description, xacro)
@@ -78,4 +78,43 @@
       </sensor>
     </gazebo>
+    <!-- RGB camera -->
+    <gazebo reference="${prefix}kinect_rgb_frame" >
+      <sensor name="camera" type="camera">
+        <camera>
+          <horizontal_fov>1.047</horizontal_fov>
+          <image>
+            <width>320</width>
+            <height>240</height>
+          </image>
+          <clip>
+            <near>0.1</near>
+            <far>100</far>
+          </clip>
+        </camera>
+        <always_on>1</always_on>
+        <update_rate>30</update_rate>
+        <visualize>true</visualize>
+        <topic>camera</topic>
+      </sensor>
+    </gazebo>
+    <!-- depth camera -->
+    <gazebo reference="${prefix}kinect_depth_frame" >
+      <sensor name="depth_camera1" type="depth_camera">
+        <update_rate>10</update_rate>
+        <topic>depth_camera</topic>
+        <camera>
+          <horizontal_fov>1.05</horizontal_fov>
+          <image>
+            <width>256</width>
+            <height>256</height>
+            <format>R_FLOAT32</format>
+          </image>
+          <clip>
+            <near>0.1</near>
+            <far>10.0</far>
+          </clip>
+        </camera>
+      </sensor>
+    </gazebo>
   </xacro:macro>
 </robot>

File: omni_car/description/urdf/kinect.urdf.xacro (robot description, xacro)
@@ -16,7 +16,5 @@
   </link>
   <link name="${prefix}${name}_depth_frame"/>
-  <link name="${prefix}${name}_depth_optical_frame"/>
   <link name="${prefix}${name}_rgb_frame"/>
-  <link name="${prefix}${name}_rgb_optical_frame"/>
   <joint name="${prefix}base_${name}_joint" type="fixed">
     <xacro:insert_block name="origin" />
@@ -29,9 +27,4 @@
     <child link="${prefix}${name}_depth_frame" />
   </joint>
-  <joint name="${prefix}${name}_depth_optical_joint" type="fixed">
-    <origin xyz="0 0 0" rpy="${-pi/2} 0 ${-pi/2}" />
-    <parent link="${prefix}${name}_depth_frame" />
-    <child link="${prefix}${name}_depth_optical_frame" />
-  </joint>
   <joint name="${prefix}${name}_rgb_joint" type="fixed">
     <origin xyz="0 -0.012 0" rpy="0 0 0" />
@@ -39,9 +32,4 @@
     <child link="${prefix}${name}_rgb_frame" />
   </joint>
-  <joint name="${prefix}${name}_rgb_optical_joint" type="fixed">
-    <origin xyz="0 0 0" rpy="${-pi/2} 0 ${-pi/2}" />
-    <parent link="${prefix}${name}_rgb_frame" />
-    <child link="${prefix}${name}_rgb_optical_frame" />
-  </joint>
   </xacro:macro>
 </robot>

Commit message: added world stl (exported soidworks and scaled), not included to gazebo

File: omni_car/description/gazebo/omni_car.gazebo.xacro (robot description, xacro)
@@ -16,4 +16,16 @@
         <cmdTopic>omni_car_controller/cmd_vel</cmdTopic>
       </plugin>
+      <!-- /usr/share/gz/gz-sim8/worlds/mecanum_drive.sdf -->
+      <!-- <plugin filename="gz-sim-mecanum-drive-system" name="gz::sim::systems::MecanumDrive">
+        <front_left_joint>wheel_front_left_joint</front_left_joint>
+        <front_right_joint>wheel_front_right_joint</front_right_joint>
+        <back_left_joint>wheel_rear_left_joint</back_left_joint>
+        <back_right_joint>wheel_rear_right_joint</back_right_joint>
+        <wheel_separation>1.25</wheel_separation>
+        <wheelbase>1.511</wheelbase>
+        <wheel_radius>0.3</wheel_radius>
+        <min_acceleration>-5</min_acceleration>
+        <max_acceleration>5</max_acceleration>
+      </plugin> -->
     </gazebo>
     <gazebo reference="${prefix}base_link">
@@ -21,5 +33,5 @@
     </gazebo>
     <!-- Properties for wheels -->
-    <xacro:property name="wheel_mu1" value="0.0"/>
+    <xacro:property name="wheel_mu1" value="1.0"/>
     <xacro:property name="wheel_mu2" value="0.0"/>
     <xacro:property name="wheel_material" value="Gazebo/Yellow"/>

Commit message: world inside gazebo, teleop params in yaml file

File: omni_car/description/gazebo/omni_car.gazebo.xacro (robot description, xacro)
@@ -33,5 +33,5 @@
     </gazebo>
     <!-- Properties for wheels -->
-    <xacro:property name="wheel_mu1" value="1.0"/>
+    <xacro:property name="wheel_mu1" value="0.0"/>
     <xacro:property name="wheel_mu2" value="0.0"/>
     <xacro:property name="wheel_material" value="Gazebo/Yellow"/>
