Commit message: new controller from diff_drive_controller, builds, not working yet

File: omni_car/description/gazebo/omni_car.gazebo.xacro (robot description, xacro)
@@ -12,8 +12,8 @@
       <plugin filename="gz-sim-imu-system" name="gz::sim::systems::Imu"/>
       <!-- Force plugin (solution to the problem mecanum wheels) -->
-      <plugin filename="force_plugin" name="force_plugin::ForcePlugin">
+      <!-- <plugin filename="force_plugin" name="force_plugin::ForcePlugin">
         <bodyName>${prefix}base_link</bodyName>
-        <cmdTopic>omni_car_controller/cmd_vel</cmdTopic>
-      </plugin>
+        <cmdTopic>omni_drive_controller/cmd_vel_out</cmdTopic>
+      </plugin> -->
       <!-- /usr/share/gz/gz-sim8/worlds/mecanum_drive.sdf -->
       <!-- <plugin filename="gz-sim-mecanum-drive-system" name="gz::sim::systems::MecanumDrive">

File: omni_car/description/ros2_control/omni_car.ros2_control.xacro (robot description, xacro)
@@ -6,32 +6,18 @@
         <plugin>gz_ros2_control/GazeboSimSystem</plugin>
       </hardware>
-      <joint name="${prefix}wheel_front_left_joint">
-        <command_interface name="velocity">
-          <param name="min">-1</param>
-          <param name="max">1</param>
-        </command_interface>
-        <state_interface name="velocity"/>
-      </joint>
-      <joint name="${prefix}wheel_front_right_joint">
-        <command_interface name="velocity">
-          <param name="min">-1</param>
-          <param name="max">1</param>
-        </command_interface>
-        <state_interface name="velocity"/>
-      </joint>
-      <joint name="${prefix}wheel_rear_left_joint">
-        <command_interface name="velocity">
-          <param name="min">-1</param>
-          <param name="max">1</param>
-        </command_interface>
-        <state_interface name="velocity"/>
-      </joint>
-      <joint name="${prefix}wheel_rear_right_joint">
-        <command_interface name="velocity">
-          <param name="min">-1</param>
-          <param name="max">1</param>
-        </command_interface>
-        <state_interface name="velocity"/>
-      </joint>
+      <xacro:macro name="joint_ros_control_properties" params="joint_name">
+        <joint name="${joint_name}">
+          <command_interface name="velocity">
+            <param name="min">-1</param>
+            <param name="max">1</param>
+          </command_interface>
+          <state_interface name="velocity"/>
+          <state_interface name="position"/>
+        </joint>
+      </xacro:macro>
+      <xacro:joint_ros_control_properties joint_name="${prefix}wheel_front_left_joint"/>
+      <xacro:joint_ros_control_properties joint_name="${prefix}wheel_front_right_joint"/>
+      <xacro:joint_ros_control_properties joint_name="${prefix}wheel_rear_left_joint"/>
+      <xacro:joint_ros_control_properties joint_name="${prefix}wheel_rear_right_joint"/>
   </ros2_control>
   </xacro:macro>
